File: files/fabpdi-t90usb/fabpdi-t90usb_v1.1.brd (EAGLE design)
At the start: 66.5 x 42.2 mm, 28 parts, among them U1 AT90USB162A, U2 GTL2003PW, U3 AMS1117-3.3, X1 16MHz

Commit message: updated t90 design files
Parts:
- moved R11 0.15 mm to (51.5, 10.7), turned to 180 degrees
Connections:
- net N$22: no longer C6.2
Routing:
- net S$1: track 0.00 -> 217.2 mm
- net N$30: track 217.4 -> 11.3 mm
- net N$22: track 30.1 -> 18.8 mm
Changed lines of the file:
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@@
 <board>
 <plain>
-<wire x1="0" y1="0" x2="66.4972" y2="-0.02" width="0" layer="20"/>
-<wire x1="66.4972" y1="-0.02" x2="66.4772" y2="42.1896" width="0" layer="20"/>
-<wire x1="66.4772" y1="42.1896" x2="0" y2="42.1896" width="0" layer="20"/>
-<wire x1="0" y1="42.1896" x2="0" y2="0" width="0" layer="20"/>
+<wire x1="0" y1="0" x2="66.4972" y2="-0.02" width="0.8128" layer="20"/>
+<wire x1="66.4972" y1="-0.02" x2="66.4772" y2="42.1896" width="0.8128" layer="20"/>
+<wire x1="66.4772" y1="42.1896" x2="0" y2="42.1896" width="0.8128" layer="20"/>
+<wire x1="0" y1="42.1896" x2="0" y2="0" width="0.8128" layer="20"/>
 <text x="33.6296" y="31.496" size="1.016" layer="51">RST</text>
 <text x="48.8696" y="3.048" size="1.016" layer="51">HWB</text>
@@
 </element>
 <element name="R7" library="00fab" package="R1206FAB" value="49" x="35.4076" y="9.652" smashed="yes" rot="R270">
-<attribute name="NAME" x="32.8676" y="8.89" size="1.016" layer="25" ratio="15" rot="R270"/>
+<attribute name="NAME" x="32.8676" y="9.525" size="1.016" layer="25" ratio="15" rot="R270"/>
 <attribute name="VALUE" x="34.8996" y="13.97" size="1.016" layer="27" ratio="15" rot="R270"/>
 </element>
 <element name="R8" library="00fab" package="R1206FAB" value="1k" x="30.5816" y="9.652" smashed="yes" rot="R90">
-<attribute name="NAME" x="29.0576" y="6.858" size="1.016" layer="25" ratio="15" rot="R90"/>
+<attribute name="NAME" x="29.0576" y="7.493" size="1.016" layer="25" ratio="15" rot="R90"/>
 <attribute name="VALUE" x="30.8356" y="5.588" size="1.016" layer="27" ratio="15" rot="R90"/>
 </element>
 <element name="R9" library="00fab" package="R1206FAB" value="100k" x="45.1866" y="9.652" smashed="yes" rot="R270">
-<attribute name="NAME" x="46.4566" y="11.43" size="1.016" layer="25" ratio="15" rot="R270"/>
-<attribute name="VALUE" x="42.9006" y="11.43" size="1.016" layer="27" ratio="15" rot="R270"/>
+<attribute name="NAME" x="42.6466" y="9.525" size="1.016" layer="25" ratio="15" rot="R270"/>
+<attribute name="VALUE" x="44.6786" y="15.24" size="1.016" layer="27" ratio="15" rot="R270"/>
 </element>
 <element name="U$1" library="00fab" package="USB_MINI" value="USB_MINI" x="4.4196" y="20.32"/>
@@
 </element>
 <element name="X1" library="00fab" package="EFOBM" value="16MHz" x="24.1046" y="9.017"/>
-<element name="R11" library="00fab" package="R1206FAB" value="0" x="51.5366" y="10.541" smashed="yes">
-<attribute name="NAME" x="49.7586" y="11.811" size="1.016" layer="25" ratio="15"/>
-<attribute name="VALUE" x="54.3306" y="10.287" size="1.016" layer="27" ratio="15"/>
+<element name="R11" library="00fab" package="R1206FAB" value="0" x="51.4604" y="10.668" smashed="yes" rot="R180">
+<attribute name="NAME" x="51.3334" y="13.208" size="1.016" layer="25" ratio="15" rot="R180"/>
+<attribute name="VALUE" x="54.8894" y="11.176" size="1.016" layer="27" ratio="15" rot="R180"/>
 </element>
 </elements>
@@
 <wire x1="12.0396" y1="23.622" x2="16.6116" y2="23.622" width="0.381" layer="1"/>
 <wire x1="16.6116" y1="14.986" x2="16.6116" y2="23.622" width="0.381" layer="1"/>
-<wire x1="16.6116" y1="14.986" x2="15.4686" y2="14.986" width="0.381" layer="1"/>
-<wire x1="15.4686" y1="13.208" x2="15.4686" y2="14.986" width="0.381" layer="1"/>
-<wire x1="15.4686" y1="13.208" x2="15.7226" y2="10.541" width="0.381" layer="1"/>
+<wire x1="16.6116" y1="14.986" x2="15.7226" y2="14.986" width="0.381" layer="1"/>
+<wire x1="15.7226" y1="13.208" x2="15.7226" y2="14.986" width="0.381" layer="1"/>
+<wire x1="15.7226" y1="13.208" x2="15.7226" y2="10.541" width="0.381" layer="1"/>
 <wire x1="12.6746" y1="10.668" x2="12.8016" y2="10.414" width="0.381" layer="1"/>
 <wire x1="12.8016" y1="10.414" x2="12.8016" y2="13.208" width="0.381" layer="1"/>
-<wire x1="12.8016" y1="13.208" x2="15.4686" y2="13.208" width="0.381" layer="1"/>
+<wire x1="12.8016" y1="13.208" x2="15.7226" y2="13.208" width="0.381" layer="1"/>
 <wire x1="24.511" y1="17.774" x2="24.511" y2="18.574" width="0.381" layer="1"/>
 <wire x1="24.511" y1="17.774" x2="22.9616" y2="17.774" width="0.381" layer="1"/>
@@
 <signal name="N$22">
 <contactref element="U2" pad="20"/>
-<contactref element="C6" pad="2"/>
 <contactref element="R9" pad="1"/>
 <wire x1="38.2016" y1="17.395" x2="38.3318" y2="17.395" width="0.3048" layer="1"/>
 <wire x1="38.2016" y1="17.395" x2="38.2016" y2="15.24" width="0.3048" layer="1"/>
-<wire x1="57.7596" y1="5.334" x2="57.7596" y2="6.985" width="0.381" layer="1"/>
 <wire x1="38.2016" y1="15.24" x2="45.1866" y2="15.24" width="0.3048" layer="1"/>
 <wire x1="45.1866" y1="15.24" x2="45.1866" y2="11.303" width="0.3048" layer="1"/>
-<wire x1="57.7596" y1="5.334" x2="54.9656" y2="5.334" width="0.381" layer="1"/>
-<wire x1="54.9656" y1="5.334" x2="54.9656" y2="10.414" width="0.381" layer="1"/>
-<wire x1="54.9656" y1="10.414" x2="53.1876" y2="10.414" width="0.381" layer="1"/>
 <wire x1="45.3136" y1="11.43" x2="48.1076" y2="11.43" width="0.381" layer="1"/>
 <wire x1="48.1076" y1="11.43" x2="48.1076" y2="10.668" width="0.381" layer="1"/>
 <wire x1="48.1076" y1="10.668" x2="50.1396" y2="10.668" width="0.381" layer="1"/>
-<wire x1="50.1396" y1="10.668" x2="53.1876" y2="10.414" width="0" layer="19" extent="1-1"/>
 <wire x1="45.1866" y1="11.303" x2="45.3136" y2="11.43" width="0" layer="19" extent="1-1"/>
 </signal>
@@
 <wire x1="52.9336" y1="19.812" x2="52.9336" y2="19.8628" width="0.3048" layer="1"/>
 </signal>
-<signal name="N$30">
-<wire x1="0" y1="0" x2="66.4972" y2="0" width="0.1016" layer="1"/>
-<wire x1="66.4972" y1="0" x2="66.4464" y2="42.2148" width="0.1016" layer="1"/>
-<wire x1="66.4464" y1="42.2148" x2="-0.0508" y2="42.2148" width="0.1016" layer="1"/>
-<wire x1="-0.0508" y1="42.2148" x2="0" y2="0" width="0.1016" layer="1"/>
-</signal>
 <signal name="N$31">
 <contactref element="R10" pad="1"/>
@@
 <wire x1="38.2016" y1="17.526" x2="38.2016" y2="18.034" width="0.3048" layer="1"/>
 </signal>
+<signal name="N$30">
+<wire x1="53.34" y1="10.541" x2="55.245" y2="10.541" width="0.381" layer="1"/>
+<wire x1="55.245" y1="10.541" x2="55.245" y2="5.334" width="0.381" layer="1"/>
+<wire x1="55.245" y1="5.334" x2="57.785" y2="5.334" width="0.381" layer="1"/>
+<wire x1="57.785" y1="5.334" x2="57.785" y2="6.985" width="0.381" layer="1"/>
+</signal>
+<signal name="S$1">
+<wire x1="0" y1="0" x2="66.421" y2="0" width="0.1016" layer="1"/>
+<wire x1="66.421" y1="0" x2="66.421" y2="42.164" width="0.1016" layer="1"/>
+<wire x1="66.421" y1="42.164" x2="0" y2="42.164" width="0.1016" layer="1"/>
+<wire x1="0" y1="42.164" x2="0" y2="0" width="0.1016" layer="1"/>
+</signal>
 </signals>
