File: files/fabpdi-t90usb/fabpdi-t90usb_v1.1.sch (EAGLE design)
At the start: 28 parts, among them U1 AT90USB162A, U2 GTL2003PW, U3 AMS1117-3.3, X1 16MHz

Commit message: updated t90 design files
Connections:
- net N$22: now also R11.2, R9.1; no longer C6.2, R11.1
- net N$30: now also C6.2, R11.1; no longer R11.2, R9.1
Other:
- moved on the sheet: C6, R11
Changed lines of the file:
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@@
 </instance>
 <instance part="JP2" gate="A" x="182.88" y="154.94" rot="R90"/>
-<instance part="C6" gate="&gt;NAME" x="165.1" y="76.2" smashed="yes" rot="R90">
-<attribute name="NAME" x="165.735" y="76.2" size="1.778" layer="95"/>
-<attribute name="VALUE" x="170.18" y="73.66" size="1.778" layer="96" rot="R180"/>
+<instance part="C6" gate="&gt;NAME" x="165.1" y="63.5" smashed="yes" rot="R90">
+<attribute name="NAME" x="165.735" y="63.5" size="1.778" layer="95"/>
+<attribute name="VALUE" x="170.18" y="60.96" size="1.778" layer="96" rot="R180"/>
 </instance>
 <instance part="C7" gate="&gt;NAME" x="200.66" y="129.54" smashed="yes" rot="R90">
@@
 </instance>
 <instance part="SUPPLY3" gate="G$1" x="165.1" y="137.16"/>
-<instance part="GND4" gate="1" x="165.1" y="66.04"/>
+<instance part="GND4" gate="1" x="165.1" y="53.34"/>
 <instance part="GND5" gate="1" x="203.2" y="66.04"/>
 <instance part="GND6" gate="1" x="182.88" y="119.38"/>
@@
 <attribute name="VALUE" x="60.198" y="85.344" size="1.778" layer="96" rot="R180"/>
 </instance>
-<instance part="R11" gate="G$1" x="165.1" y="111.76" smashed="yes" rot="R90">
-<attribute name="NAME" x="163.83" y="115.3414" size="1.778" layer="95" rot="R180"/>
-<attribute name="VALUE" x="162.306" y="110.998" size="1.778" layer="96" rot="R180"/>
+<instance part="R11" gate="G$1" x="165.1" y="73.66" smashed="yes" rot="R90">
+<attribute name="NAME" x="163.83" y="77.2414" size="1.778" layer="95" rot="R180"/>
+<attribute name="VALUE" x="162.306" y="72.898" size="1.778" layer="96" rot="R180"/>
 </instance>
 </instances>
@@
 <pinref part="C6" gate="&gt;NAME" pin="1"/>
 <pinref part="GND4" gate="1" pin="GND"/>
-<wire x1="165.1" y1="71.12" x2="165.1" y2="68.58" width="0.1524" layer="91"/>
+<wire x1="165.1" y1="58.42" x2="165.1" y2="55.88" width="0.1524" layer="91"/>
 </segment>
 <segment>
@@
 <segment>
 <pinref part="U2" gate="G$1" pin="GREF"/>
-<pinref part="C6" gate="&gt;NAME" pin="2"/>
 <wire x1="170.18" y1="81.28" x2="165.1" y2="81.28" width="0.1524" layer="91"/>
-<wire x1="165.1" y1="81.28" x2="165.1" y2="78.74" width="0.1524" layer="91"/>
-<junction x="165.1" y="81.28"/>
 <pinref part="U2" gate="G$1" pin="DREF"/>
 <wire x1="165.1" y1="83.82" x2="165.1" y2="81.28" width="0.1524" layer="91"/>
 <wire x1="170.18" y1="83.82" x2="165.1" y2="83.82" width="0.1524" layer="91"/>
-<pinref part="R11" gate="G$1" pin="1"/>
-<wire x1="165.1" y1="106.68" x2="165.1" y2="83.82" width="0.1524" layer="91"/>
+<pinref part="R9" gate="G$1" pin="1"/>
+<wire x1="165.1" y1="119.38" x2="165.1" y2="83.82" width="0.1524" layer="91"/>
 <junction x="165.1" y="83.82"/>
+<pinref part="R11" gate="G$1" pin="2"/>
+<wire x1="165.1" y1="81.28" x2="165.1" y2="78.74" width="0.1524" layer="91"/>
+<junction x="165.1" y="81.28"/>
 </segment>
 </net>
@@
 <net name="N$30" class="0">
 <segment>
-<pinref part="R9" gate="G$1" pin="1"/>
-<pinref part="R11" gate="G$1" pin="2"/>
-<wire x1="165.1" y1="119.38" x2="165.1" y2="116.84" width="0.1524" layer="91"/>
-</segment>
-</net>
+<pinref part="R11" gate="G$1" pin="1"/>
+<pinref part="C6" gate="&gt;NAME" pin="2"/>
+<wire x1="165.1" y1="68.58" x2="165.1" y2="66.04" width="0.1524" layer="91"/>
+</segment>
+</net>
