File: files/fabpdi-t90usb/fabpdi-t90usb_v1.brd (EAGLE design)
At the start: 71.1 x 42.9 mm, 28 parts, among them U1 AT90USB162A, U2 GTL2003PW, U3 AMS1117-3.3, X1 16MHz

Commit message: updated t90 design files
Parts:
- R11: device 00fab:LED1206FAB -> 00fab:R1206FAB
Routing:
- net S$1: track 80.4 -> 77.4 mm
- net S$2: track 0.00 -> 2.79 mm
- net N$22: track 112.1 -> 112.7 mm
Changed lines of the file:
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@@
 <setting verticaltext="up"/>
 </settings>
-<grid distance="0.01" unitdist="inch" unit="inch" style="lines" multiple="4" display="yes" altdistance="0.005" altunitdist="inch" altunit="inch"/>
+<grid distance="0.01" unitdist="inch" unit="inch" style="lines" multiple="4" display="no" altdistance="0.005" altunitdist="inch" altunit="inch"/>
 <layers>
 <layer number="1" name="Top" color="4" fill="1" visible="yes" active="yes"/>
@@
 <layer number="17" name="Pads" color="2" fill="1" visible="yes" active="yes"/>
 <layer number="18" name="Vias" color="2" fill="1" visible="yes" active="yes"/>
-<layer number="19" name="Unrouted" color="6" fill="1" visible="yes" active="yes"/>
+<layer number="19" name="Unrouted" color="6" fill="1" visible="no" active="yes"/>
 <layer number="20" name="Dimension" color="15" fill="1" visible="yes" active="yes"/>
 <layer number="21" name="tPlace" color="7" fill="1" visible="yes" active="yes"/>
 <layer number="22" name="bPlace" color="7" fill="1" visible="no" active="yes"/>
-<layer number="23" name="tOrigins" color="15" fill="1" visible="yes" active="yes"/>
+<layer number="23" name="tOrigins" color="15" fill="1" visible="no" active="yes"/>
 <layer number="24" name="bOrigins" color="15" fill="1" visible="no" active="yes"/>
 <layer number="25" name="tNames" color="7" fill="1" visible="yes" active="yes"/>
@@
 <board>
 <plain>
-<wire x1="0" y1="0" x2="71.12" y2="-0.02" width="0" layer="20"/>
-<wire x1="71.12" y1="-0.02" x2="71.1" y2="42.85" width="0" layer="20"/>
-<wire x1="71.1" y1="42.85" x2="0" y2="42.85" width="0" layer="20"/>
-<wire x1="0" y1="42.85" x2="0" y2="0" width="0" layer="20"/>
+<wire x1="0" y1="0" x2="71.12" y2="-0.02" width="0.8128" layer="20"/>
+<wire x1="71.12" y1="-0.02" x2="71.1" y2="42.85" width="0.8128" layer="20"/>
+<wire x1="71.1" y1="42.85" x2="0" y2="42.85" width="0.8128" layer="20"/>
+<wire x1="0" y1="42.85" x2="0" y2="0" width="0.8128" layer="20"/>
 <text x="34.29" y="31.496" size="1.016" layer="51">RST</text>
 <text x="49.53" y="3.048" size="1.016" layer="51">HWB</text>
@@
 </element>
 <element name="X1" library="00fab" package="EFOBM" value="16MHz" x="24.765" y="8.255"/>
-<element name="R11" library="00fab" package="LED1206FAB" value="0" x="46.228" y="12.954" smashed="yes" rot="R90">
+<element name="R11" library="00fab" package="R1206FAB" value="0" x="46.228" y="12.954" smashed="yes" rot="R90">
 <attribute name="NAME" x="44.704" y="10.16" size="1.016" layer="25" ratio="15" rot="R90"/>
 <attribute name="VALUE" x="48.514" y="14.478" size="1.016" layer="27" ratio="15" rot="R90"/>
@@
 <wire x1="49.53" y1="30.734" x2="47.625" y2="30.734" width="0.381" layer="1"/>
 <contactref element="JP5" pad="2"/>
-<wire x1="46.228" y1="14.478" x2="46.193378125" y2="14.478" width="0.381" layer="1"/>
 <wire x1="48.768" y1="17.395" x2="48.768" y2="16.764" width="0.3048" layer="1"/>
-<wire x1="46.193378125" y1="17.395" x2="48.768" y2="17.395" width="0.3048" layer="1"/>
-<wire x1="46.193378125" y1="14.478" x2="46.193378125" y2="17.395" width="0.381" layer="1"/>
+<wire x1="44.8278" y1="17.395" x2="48.768" y2="17.395" width="0.3048" layer="1"/>
 <wire x1="35.941" y1="28.702" x2="35.941" y2="34.671" width="0.381" layer="1"/>
 <wire x1="49.53" y1="28.702" x2="49.53" y2="30.734" width="0.381" layer="1"/>
@@
 <wire x1="40.64" y1="28.702" x2="35.941" y2="28.702" width="0.381" layer="1"/>
 <contactref element="U2" pad="1"/>
-<wire x1="46.193378125" y1="17.395" x2="44.8278" y2="17.395" width="0.3048" layer="1"/>
 <wire x1="40.64" y1="17.395" x2="44.8278" y2="17.395" width="0.3048" layer="1"/>
 <wire x1="40.64" y1="17.395" x2="40.64" y2="28.702" width="0.3048" layer="1"/>
@@
 <wire x1="28.194" y1="7.62" x2="33.782" y2="7.62" width="0.381" layer="1"/>
 <wire x1="33.782" y1="7.62" x2="33.782" y2="3.683" width="0.381" layer="1"/>
-<wire x1="33.782" y1="3.683" x2="46.255071875" y2="3.683" width="0.381" layer="1"/>
-<wire x1="46.255071875" y1="3.683" x2="46.255071875" y2="11.43" width="0.381" layer="1"/>
-<wire x1="46.228" y1="14.478" x2="46.255071875" y2="14.478" width="0.381" layer="16"/>
-<wire x1="46.255071875" y1="14.478" x2="46.255071875" y2="11.43" width="0" layer="19" extent="1-16"/>
+<wire x1="46.228" y1="3.683" x2="46.228" y2="11.43" width="0.381" layer="1"/>
+<wire x1="33.782" y1="3.683" x2="46.228" y2="3.683" width="0.381" layer="1"/>
 <wire x1="28.194" y1="4.318" x2="28.194" y2="7.62" width="0" layer="19" extent="1-1"/>
 </signal>
@@
 <contactref element="R9" pad="1"/>
 <wire x1="38.9922" y1="17.395" x2="38.862" y2="17.395" width="0.3048" layer="1"/>
-<wire x1="38.862" y1="17.395" x2="38.862" y2="12.954" width="0.3048" layer="1"/>
+<wire x1="38.862" y1="17.395" x2="38.862" y2="17.272" width="0.3048" layer="1"/>
+<wire x1="38.862" y1="17.272" x2="38.862" y2="12.954" width="0.3048" layer="1"/>
 <wire x1="38.862" y1="12.954" x2="50.927" y2="12.954" width="0.3048" layer="1"/>
 <wire x1="50.927" y1="12.954" x2="50.927" y2="4.064" width="0.3048" layer="1"/>
@@
 <wire x1="56.007" y1="32.131" x2="60.5028" y2="32.131" width="0.3048" layer="1"/>
 <wire x1="60.5028" y1="32.131" x2="60.5028" y2="28.956" width="0.381" layer="1"/>
+<wire x1="38.862" y1="17.395" x2="38.862" y2="18.034" width="0.3048" layer="1"/>
 </signal>
 <signal name="N$24">
@@
 <wire x1="26.115" y1="11.938" x2="26.115" y2="8.255" width="0.381" layer="1"/>
 </signal>
+<signal name="S$2">
+<wire x1="46.228" y1="14.478" x2="46.228" y2="17.272" width="0.381" layer="1"/>
+</signal>
 </signals>
