File: files/fabpdi-t90usb/fabpdi-t90usb_v1.sch (EAGLE design)
At the start: 27 parts, among them U1 AT90USB162A, U2 GTL2003PW, U3 AMS1117-3.3, X1 16MHz

Commit message: updated t90 design files
Parts:
- added R11: 0, 00fab:RES-US1206FAB
Connections:
- new net GND': C6.1, C7.1, JP3.6, JP4.6, R11.2, U2.GND
- net GND: now also R11.1; no longer C6.1, C7.1, JP3.6, JP4.6, U2.GND
- net N$22: now also U2.DREF
Changed lines of the file:
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@@
 <part name="U3" library="Seeed-IC" library_urn="urn:adsk.eagle:library:470" deviceset="PMIC-CJT1117-3.3(SOT223)" device="" value="AMS1117-3.3"/>
 <part name="SUPPLY3" library="SparkFun-Aesthetics" deviceset="VCC" device=""/>
-<part name="GND4" library="SparkFun-Aesthetics" deviceset="GND" device=""/>
-<part name="GND5" library="SparkFun-Aesthetics" deviceset="GND" device=""/>
+<part name="GND4" library="SparkFun-Aesthetics" deviceset="GND" device="" value="GND*"/>
+<part name="GND5" library="SparkFun-Aesthetics" deviceset="GND" device="" value="GND*"/>
 <part name="GND6" library="SparkFun-Aesthetics" deviceset="GND" device=""/>
-<part name="GND7" library="SparkFun-Aesthetics" deviceset="GND" device=""/>
+<part name="GND7" library="SparkFun-Aesthetics" deviceset="GND" device="" value="GND*"/>
 <part name="V+" library="supply2" library_urn="urn:adsk.eagle:library:372" deviceset="VCC" device="" value="V+"/>
 <part name="SUPPLY5" library="supply2" library_urn="urn:adsk.eagle:library:372" deviceset="VCC" device="" value="V+"/>
@@
 <part name="R10" library="00fab" deviceset="RES-US" device="1206FAB" value="0"/>
 <part name="X1" library="00fab" deviceset="RESONATOR" device="" value="16MHz"/>
+<part name="GND8" library="supply1" library_urn="urn:adsk.eagle:library:371" deviceset="GND" device="" value="GND*"/>
+<part name="R11" library="00fab" deviceset="RES-US" device="1206FAB" value="0"/>
 </parts>
 <sheets>
@@
 <attribute name="NAME" x="54.864" y="95.758" size="1.778" layer="95"/>
 <attribute name="VALUE" x="60.198" y="85.344" size="1.778" layer="96" rot="R180"/>
+</instance>
+<instance part="GND8" gate="1" x="200.66" y="119.38"/>
+<instance part="R11" gate="G$1" x="190.5" y="121.92" smashed="yes">
+<attribute name="NAME" x="188.468" y="123.6726" size="1.778" layer="95"/>
+<attribute name="VALUE" x="189.23" y="118.618" size="1.778" layer="96"/>
 </instance>
 </instances>
@@
 </segment>
 <segment>
+<pinref part="GND6" gate="1" pin="GND"/>
 <pinref part="U3" gate="G$1" pin="GND"/>
-<pinref part="GND6" gate="1" pin="GND"/>
 <wire x1="182.88" y1="124.46" x2="182.88" y2="121.92" width="0.1524" layer="91"/>
-<pinref part="C7" gate="&gt;NAME" pin="1"/>
-<wire x1="200.66" y1="124.46" x2="200.66" y2="121.92" width="0.1524" layer="91"/>
-<wire x1="200.66" y1="121.92" x2="182.88" y2="121.92" width="0.1524" layer="91"/>
+<pinref part="R11" gate="G$1" pin="1"/>
+<wire x1="185.42" y1="121.92" x2="182.88" y2="121.92" width="0.1524" layer="91"/>
 <junction x="182.88" y="121.92"/>
-</segment>
-<segment>
-<pinref part="U2" gate="G$1" pin="GND"/>
-<pinref part="GND5" gate="1" pin="GND"/>
-<wire x1="200.66" y1="81.28" x2="203.2" y2="81.28" width="0.1524" layer="91"/>
-<wire x1="203.2" y1="81.28" x2="203.2" y2="68.58" width="0.1524" layer="91"/>
-</segment>
-<segment>
-<pinref part="C6" gate="&gt;NAME" pin="1"/>
-<pinref part="GND4" gate="1" pin="GND"/>
-<wire x1="165.1" y1="71.12" x2="165.1" y2="68.58" width="0.1524" layer="91"/>
-</segment>
-<segment>
-<pinref part="JP3" gate="A" pin="6"/>
-<pinref part="GND7" gate="1" pin="GND"/>
-<wire x1="233.68" y1="106.68" x2="243.84" y2="106.68" width="0.1524" layer="91"/>
-<wire x1="243.84" y1="106.68" x2="243.84" y2="91.44" width="0.1524" layer="91"/>
-<pinref part="JP4" gate="A" pin="6"/>
-<wire x1="243.84" y1="91.44" x2="243.84" y2="83.82" width="0.1524" layer="91"/>
-<wire x1="233.68" y1="91.44" x2="243.84" y2="91.44" width="0.1524" layer="91"/>
-<junction x="243.84" y="91.44"/>
 </segment>
 </net>
@@
 <wire x1="165.1" y1="81.28" x2="165.1" y2="78.74" width="0.1524" layer="91"/>
 <pinref part="R9" gate="G$1" pin="1"/>
-<wire x1="165.1" y1="114.3" x2="165.1" y2="81.28" width="0.1524" layer="91"/>
+<wire x1="165.1" y1="114.3" x2="165.1" y2="83.82" width="0.1524" layer="91"/>
 <junction x="165.1" y="81.28"/>
+<pinref part="U2" gate="G$1" pin="DREF"/>
+<wire x1="165.1" y1="83.82" x2="165.1" y2="81.28" width="0.1524" layer="91"/>
+<wire x1="170.18" y1="83.82" x2="165.1" y2="83.82" width="0.1524" layer="91"/>
+<junction x="165.1" y="83.82"/>
 </segment>
 </net>
@@
 </segment>
 </net>
+<net name="GND'" class="0">
+<segment>
+<pinref part="C6" gate="&gt;NAME" pin="1"/>
+<pinref part="GND4" gate="1" pin="GND"/>
+<wire x1="165.1" y1="71.12" x2="165.1" y2="68.58" width="0.1524" layer="91"/>
+</segment>
+<segment>
+<pinref part="U2" gate="G$1" pin="GND"/>
+<pinref part="GND5" gate="1" pin="GND"/>
+<wire x1="200.66" y1="81.28" x2="203.2" y2="81.28" width="0.1524" layer="91"/>
+<wire x1="203.2" y1="81.28" x2="203.2" y2="68.58" width="0.1524" layer="91"/>
+</segment>
+<segment>
+<pinref part="C7" gate="&gt;NAME" pin="1"/>
+<pinref part="GND8" gate="1" pin="GND"/>
+<wire x1="200.66" y1="124.46" x2="200.66" y2="121.92" width="0.1524" layer="91"/>
+<pinref part="R11" gate="G$1" pin="2"/>
+<wire x1="195.58" y1="121.92" x2="200.66" y2="121.92" width="0.1524" layer="91"/>
+<junction x="200.66" y="121.92"/>
+</segment>
+<segment>
+<pinref part="JP3" gate="A" pin="6"/>
+<pinref part="GND7" gate="1" pin="GND"/>
+<wire x1="233.68" y1="106.68" x2="243.84" y2="106.68" width="0.1524" layer="91"/>
+<wire x1="243.84" y1="106.68" x2="243.84" y2="91.44" width="0.1524" layer="91"/>
+<pinref part="JP4" gate="A" pin="6"/>
+<wire x1="243.84" y1="91.44" x2="243.84" y2="83.82" width="0.1524" layer="91"/>
+<wire x1="233.68" y1="91.44" x2="243.84" y2="91.44" width="0.1524" layer="91"/>
+<junction x="243.84" y="91.44"/>
+</segment>
+</net>
 </nets>
 </sheet>
 </sheets>
+<errors>
+</errors>
 </schematic>
 </drawing>
